File: ErnoCCC-Kicad/PCB-Negative.kicad_pcb (KiCad board)
At the start: 2 copper layers, 197 x 137 mm, 0 parts

Commit message: Trying to fix the missing solder mask on the stencil board probably still needs a net though
Other:
- board text added: "Bottom"
- board text added: "Erno Crystal Counter Controller"
Changed lines of the file:
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@@
   (general
     (thickness 1.6)
-    (drawings 51)
+    (drawings 53)
     (tracks 0)
     (zones 0)
@@
     (uvia_drill 0.1)
   )
+  (gr_text Bottom (at 149.5 149) (layer B.Mask)
+    (effects (font (size 3 3) (thickness 0.5)) (justify mirror))
+  )
+  (gr_text "Erno\nCrystal Counter Controller" (at 87 148.2) (layer F.Mask)
+    (effects (font (size 3 3) (thickness 0.6)))
+  )
   (gr_arc (start 214.7 101.1) (end 215.5 101) (angle -137.3373059) (layer Edge.Cuts) (width 0.05))
